Commit message: Added Gazebo simulation. Tested w movement

File: src/my_robot_description/urdf/my_robot.urdf (robot description, URDF)
Before this commit: robot my_robot, 3 links, 2 joints
Links:
- link base_link: mass None -> 0.5
Joints:
- joint left_wheel_joint: axis 0 1 0 -> 0 0 1
- joint right_wheel_joint: axis 0 1 0 -> 0 0 1
